File: extension.brd (EAGLE design)
At the start: 144.8 x 48.3 mm, 2 parts

Commit message: route all wires
Routing:
- net 3: track 0.00 -> 56.9 mm
- net 32: track 0.00 -> 55.8 mm
- net 1: track 0.00 -> 55.8 mm
- net 9: track 0.00 -> 55.8 mm
- net 8: track 0.00 -> 55.8 mm
- net 7: track 0.00 -> 55.8 mm
- net 6: track 0.00 -> 55.8 mm
- net 5: track 0.00 -> 55.8 mm
- net 4: track 0.00 -> 55.8 mm
- net 31: track 0.00 -> 55.8 mm
- net 30: track 0.00 -> 55.8 mm
- net 29: track 0.00 -> 55.8 mm
- net 28: track 0.00 -> 55.8 mm
- net 27: track 0.00 -> 55.8 mm
- net 26: track 0.00 -> 55.8 mm
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